File: yoring.kicad_sch (KiCad schematic)
At the start: 65 parts, among them J1 USB-C_USB4105-GF-A, J3 Conn_01x05, SW1 SW_MEC_5E, SW2 SW_MEC_5E, U1 ESP32C3, U2 IS25LP016D-JLLE, U4 ICM-20602, U4 USBLC6-2SC6, U5 ICM-20602, U6 ICM-20602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

Commit message: Commit before local repo deletion
Parts:
- renumbered C17 to C1, C17 to C11, C17 to C12, C17 to C13, C17 to C14, C17 to C15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
